Commit message: sailboat loading in vrx scenario

File: sailboat_gazebo/urdf/dynamics/sailboat_gazebo_dynamics_plugin.xacro (robot description, xacro)
@@ -1,6 +1,6 @@
 <?xml version="1.0"?>
 <robot xmlns:xacro="http://ros.org/wiki/xacro">
-  <xacro:macro name="usv_dynamics_gazebo" params="name">
-    <!--Gazebo Plugin for simulating Sailboat dynamics-->
+  <xacro:macro name="usv_dynamics_gazebo" params="name width:=1.2 length:=2">
+    <!--Gazebo Plugin for simulating WAM-V dynamics-->
     <gazebo>
       <plugin name="usv_dynamics_${name}" filename="libusv_gazebo_dynamics_plugin.so">
@@ -25,20 +25,11 @@
         <!-- General dimensions -->
         <!--<boatArea>2.2</boatArea>-->
-		<hullRadius>0.213</hullRadius>
-        <boatWidth>2.4</boatWidth>
-        <boatLength>4.9</boatLength>
-		<!-- Length discretization, AKA, "N" -->
-		<length_n>2</length_n>
-        <!-- Waves x3 -->
-        <wave_n>3</wave_n>
-        <wave_amp0>0.06</wave_amp0>
-        <wave_period0>12.6</wave_period0>
-        <wave_direction0>-1 0</wave_direction0>
-        <wave_amp1>0.04</wave_amp1>
-        <wave_period1>3.7</wave_period1>
-        <wave_direction1>-0.7 0.7</wave_direction1>
-        <wave_amp2>0.03</wave_amp2>
-        <wave_period2>6.3</wave_period2>
-        <wave_direction2>0.7 0.7</wave_direction2>
+        <hullRadius>0.213</hullRadius>
+        <boatWidth>${width}</boatWidth>
+        <boatLength>${length}</boatLength>
+        <!-- Length discretization, AKA, "N" -->
+        <length_n>2</length_n>
+        <!-- Wave model -->
+        <wave_model>ocean_waves</wave_model>
       </plugin>
     </gazebo>

File: sailboat_gazebo/urdf/sailboat_gazebo.urdf.xacro (robot description, xacro)
@@ -9,5 +9,5 @@
   <xacro:arg name="ground_truth_enabled" default="false" />
   <xacro:arg name="vrx_sensors_enabled" default="false" />
-  <!-- === The WAM-V platform === -->
+  <!-- === The sailboat platform === -->
   <xacro:include filename="$(find sailboat_gazebo)/urdf/sailboat_gazebo.xacro" />
   <!-- Add a front camera -->

File: sailboat_gazebo/urdf/sailboat_gazebo.xacro (robot description, xacro)
@@ -8,4 +8,4 @@
   <xacro:usv_dynamics_gazebo name="sailboat_dynamics_plugin"/>
   <!-- Attach wind plugin -->
-  <xacro:usv_wind_gazebo name="sailboat_wind_plugin"/>
+  <!--<xacro:usv_wind_gazebo name="sailboat_wind_plugin"/>-->
 </robot>
