Commit message: added sail stl

File: sailboat_description/urdf/sailboat_base.urdf.xacro (robot description, xacro)
@@ -81,7 +81,7 @@
 	    </collision>
 	    <visual name="visual">
-            <geometry>
-              <box size="0.4 0.02 1" />
-            </geometry>
+          <geometry>
+            <mesh filename="package://sailboat_description/mesh/sail.stl"/>
+          </geometry>
             <origin rpy="0 0 0" xyz="0 0 0"/>
 	    </visual>

Commit message: added sail stl

File: sailboat_description/urdf/sailboat_base.urdf.xacro (robot description, xacro)
@@ -82,5 +82,5 @@
 	    <visual name="visual">
           <geometry>
-            <mesh filename="package://sailboat_description/mesh/sail.stl"/>
+            <mesh filename="package://sailboat_description/mesh/sail.dae"/>
           </geometry>
             <origin rpy="0 0 0" xyz="0 0 0"/>

Commit message: fixed boat scale with real model

File: sailboat_description/urdf/sailboat_base.urdf.xacro (robot description, xacro)
@@ -5,5 +5,5 @@
     <link name="base_link">
         <visual>
-          <origin rpy="1.57079632679 0 1.57079632679"/>
+          <origin rpy="0 0 0"/>
           <geometry>
             <mesh filename="package://sailboat_description/mesh/pt90.stl"/>
@@ -12,5 +12,5 @@
         </visual>
         <collision>
-          <origin rpy="1.57079632679 0 1.57079632679"/>
+          <origin rpy="0 0 0"/>
           <geometry>
             <mesh filename="package://sailboat_description/mesh/pt90.stl"/>
@@ -18,5 +18,5 @@
         </collision>
         <inertial>
-            <origin rpy="0 0 0" xyz="0 0 -0.05"/>
+          <origin rpy="0 0 0" xyz="0 0 -0.05"/>
           <mass value="10"/>
           <inertia ixx="0.1" ixy="0.0" ixz="0.0" iyy="1.4" iyz="0.0" izz="1.4"/>
@@ -76,7 +76,7 @@
 	    <collision name="collision">
             <geometry>
-              <box size="0.4 0.02 1" />
+              <mesh filename="package://sailboat_description/mesh/sail.dae"/>
             </geometry>
-            <origin rpy="0 0 0" xyz="0 0 0"/>
+            <origin rpy="0 0 0" xyz="0.4 0 0.6"/>
 	    </collision>
 	    <visual name="visual">
@@ -84,5 +84,5 @@
             <mesh filename="package://sailboat_description/mesh/sail.dae"/>
           </geometry>
-            <origin rpy="0 0 0" xyz="0 0 0"/>
+            <origin rpy="0 0 0" xyz="0.4 0 0.6"/>
 	    </visual>
     </link>
@@ -90,8 +90,40 @@
         <parent link="base_link"/>
         <child link="sail"/>
-        <origin rpy="0 0 ${PI/2}" xyz="0 0 +0.6"/>
+        <origin rpy="0 0 0" xyz="0.4 0 0.6"/>
         <dynamics damping="1.0"/>
         <axis xyz="0 0 1"/>
         <limit effort="30" velocity="5" lower="-${PI/2}" upper="${PI/2}" />
     </joint>
+    <!-- KEEL DESCRIPTION -->
+    <link name="keel">
+        <inertial>
+            <mass value="0.05" />
+            <inertia
+              ixx="0.05"
+              ixy="0.0"
+              iyy="0.05"
+              ixz="0.0"
+              iyz="0.0"
+              izz="0.005"/>
+        </inertial>
+        <collision name="collision">
+            <geometry>
+              <mesh filename="package://sailboat_description/mesh/keel.stl"/>
+            </geometry>
+            <origin rpy="0 0 0" xyz="0 0 -0.5"/>
+        </collision>
+        <visual name="visual">
+            <geometry>
+              <mesh filename="package://sailboat_description/mesh/keel.stl"/>
+            </geometry>
+            <origin rpy="0 0 0" xyz="0 0 0"/>
+        </visual>
+    </link>
+    <joint name="keel_joint" type="revolute">
+        <parent link="base_link"/>
+        <child link="keel"/>
+        <origin rpy="0 0 0" xyz="-0.53 0 -0.1"/>
+        <axis xyz="0 0 1"/>
+        <limit effort="50" velocity="5" lower="0" upper="0" />
+    </joint>
 </robot>

Commit message: added rudder

File: sailboat_description/urdf/sailboat_base.urdf.xacro (robot description, xacro)
@@ -19,13 +19,7 @@
         <inertial>
           <origin rpy="0 0 0" xyz="0 0 -0.05"/>
-          <mass value="10"/>
+          <mass value="0.5"/>
           <inertia ixx="0.1" ixy="0.0" ixz="0.0" iyy="1.4" iyz="0.0" izz="1.4"/>
         </inertial>
-        <buoyancy>
-          <compensation>1.2</compensation>
-          <origin xyz="-0.0005 0 0.05"/>
-          <limit radius="0.1"/>
-          <damping rpy="20 50 50" xyz="20 50 50"/>
-        </buoyancy>
     </link>
     <!-- RUDDER DESCRIPTION -->
@@ -43,13 +37,13 @@
             <collision name="collision">
                 <geometry>
-                  <box size="0.1 0.02 0.3" />
+                  <mesh filename="package://sailboat_description/mesh/rudder.stl"/>
                 </geometry>
-                <origin rpy="0 0 0" xyz="-0.1 0 0"/>
+                <origin rpy="0 0 0" xyz="-0.2 0 0"/>
             </collision>
             <visual name="visual">
                 <geometry>
-                  <box size="0.1 0.02 0.3" />
+                  <mesh filename="package://sailboat_description/mesh/rudder.stl"/>
                 </geometry>
-                <origin rpy="0 0 0" xyz="-0.1 0 0"/>
+                <origin rpy="0 0 0" xyz="-0.2 0 0"/>
             </visual>
         </link>
@@ -57,5 +51,5 @@
             <parent link="base_link"/>
             <child link="rudder"/>
-            <origin rpy="0 0 0" xyz="-0.53 0 -0.1"/>
+            <origin rpy="0 0 0" xyz="-0.2 0 0.0"/>
             <dynamics damping="1.0"/>
             <axis xyz="0 0 1"/>
@@ -78,5 +72,5 @@
               <mesh filename="package://sailboat_description/mesh/sail.dae"/>
             </geometry>
-            <origin rpy="0 0 0" xyz="0.4 0 0.6"/>
+            <origin rpy="0 0 0" xyz="0.05 0 0.0"/>
 	    </collision>
 	    <visual name="visual">
@@ -84,5 +78,5 @@
             <mesh filename="package://sailboat_description/mesh/sail.dae"/>
           </geometry>
-            <origin rpy="0 0 0" xyz="0.4 0 0.6"/>
+            <origin rpy="0 0 0" xyz="0.05 0 0.0"/>
 	    </visual>
     </link>
@@ -90,5 +84,5 @@
         <parent link="base_link"/>
         <child link="sail"/>
-        <origin rpy="0 0 0" xyz="0.4 0 0.6"/>
+        <origin rpy="0 0 0" xyz="0.05 0 0.0"/>
         <dynamics damping="1.0"/>
         <axis xyz="0 0 1"/>
@@ -111,5 +105,5 @@
               <mesh filename="package://sailboat_description/mesh/keel.stl"/>
             </geometry>
-            <origin rpy="0 0 0" xyz="0 0 -0.5"/>
+            <origin rpy="0 0 0" xyz="0 0 0"/>
         </collision>
         <visual name="visual">
@@ -123,5 +117,5 @@
         <parent link="base_link"/>
         <child link="keel"/>
-        <origin rpy="0 0 0" xyz="-0.53 0 -0.1"/>
+        <origin rpy="0 0 0" xyz="0 0 0.0"/>
         <axis xyz="0 0 1"/>
         <limit effort="50" velocity="5" lower="0" upper="0" />

Commit message: added teleop control at sailboat_teleop

File: sailboat_description/urdf/sailboat_base.urdf.xacro (robot description, xacro)
@@ -39,5 +39,5 @@
                   <mesh filename="package://sailboat_description/mesh/rudder.stl"/>
                 </geometry>
-                <origin rpy="0 0 0" xyz="-0.2 0 0"/>
+                <origin rpy="0 0 0" xyz="0.0 0 0"/>
             </collision>
             <visual name="visual">
@@ -45,5 +45,5 @@
                   <mesh filename="package://sailboat_description/mesh/rudder.stl"/>
                 </geometry>
-                <origin rpy="0 0 0" xyz="-0.2 0 0"/>
+                <origin rpy="0 0 0" xyz="0.0 0 0"/>
             </visual>
         </link>
@@ -51,5 +51,5 @@
             <parent link="base_link"/>
             <child link="rudder"/>
-            <origin rpy="0 0 0" xyz="-0.2 0 0.0"/>
+            <origin rpy="0 0 0" xyz="-0.4 0 0.0"/>
             <dynamics damping="1.0"/>
             <axis xyz="0 0 1"/>
@@ -72,5 +72,5 @@
               <mesh filename="package://sailboat_description/mesh/sail.dae"/>
             </geometry>
-            <origin rpy="0 0 0" xyz="0.05 0 0.0"/>
+            <origin rpy="0 0 0" xyz="0.0 0 0.0"/>
 	    </collision>
 	    <visual name="visual">
@@ -78,5 +78,5 @@
             <mesh filename="package://sailboat_description/mesh/sail.dae"/>
           </geometry>
-            <origin rpy="0 0 0" xyz="0.05 0 0.0"/>
+            <origin rpy="0 0 0" xyz="0.0 0 0.0"/>
 	    </visual>
     </link>
@@ -84,40 +84,31 @@
         <parent link="base_link"/>
         <child link="sail"/>
-        <origin rpy="0 0 0" xyz="0.05 0 0.0"/>
+        <origin rpy="0 0 0" xyz="0.25 0 0.0"/>
         <dynamics damping="1.0"/>
         <axis xyz="0 0 1"/>
         <limit effort="30" velocity="5" lower="-${PI/2}" upper="${PI/2}" />
     </joint>
-    <!-- KEEL DESCRIPTION -->
-    <link name="keel">
-        <inertial>
-            <mass value="0.05" />
-            <inertia
-              ixx="0.05"
-              ixy="0.0"
-              iyy="0.05"
-              ixz="0.0"
-              iyz="0.0"
-              izz="0.005"/>
-        </inertial>
-        <collision name="collision">
-            <geometry>
-              <mesh filename="package://sailboat_description/mesh/keel.stl"/>
-            </geometry>
-            <origin rpy="0 0 0" xyz="0 0 0"/>
-        </collision>
-        <visual name="visual">
-            <geometry>
-              <mesh filename="package://sailboat_description/mesh/keel.stl"/>
-            </geometry>
-            <origin rpy="0 0 0" xyz="0 0 0"/>
-        </visual>
-    </link>
-    <joint name="keel_joint" type="revolute">
-        <parent link="base_link"/>
-        <child link="keel"/>
-        <origin rpy="0 0 0" xyz="0 0 0.0"/>
-        <axis xyz="0 0 1"/>
-        <limit effort="50" velocity="5" lower="0" upper="0" />
+  <gazebo>
+    <plugin name="gazebo_ros_control" filename="libgazebo_ros_control.so">
+      <robotNamespace>/sailboat</robotNamespace>
+    </plugin>
+  </gazebo>
+  <transmission name="sail_trans">
+    <type>transmission_interface/SimpleTransmission</type>
+    <actuator name="sail_act">
+      <mechanicalReduction>1</mechanicalReduction>
+    </actuator>
+    <joint name="sail_joint">
+      <hardwareInterface>hardware_interface/PositionJointInterface</hardwareInterface>
     </joint>
+  </transmission>
+  <transmission name="rudder_trans">
+    <type>transmission_interface/SimpleTransmission</type>
+    <actuator name="rudder_act">
+      <mechanicalReduction>1</mechanicalReduction>
+    </actuator>
+    <joint name="rudder_joint">
+      <hardwareInterface>hardware_interface/PositionJointInterface</hardwareInterface>
+    </joint>
+  </transmission>
 </robot>

Commit message: fixed sailboat model

File: sailboat_description/urdf/sailboat_base.urdf.xacro (robot description, xacro)
@@ -2,8 +2,9 @@
 <robot name="sailboat" xmlns:xacro="http://www.ros.org/wiki/xacro">
     <xacro:property name="PI" value="3.1415926535897931"/>
+    <xacro:property name="disp" value="0.0"/>
     <!-- HULL DESCRIPTION -->
     <link name="base_link">
         <visual>
-          <origin rpy="0 0 0"/>
+          <origin rpy="0 0 0" xyz="0 0 ${disp}"/>
           <geometry>
             <mesh filename="package://sailboat_description/mesh/pt90.stl"/>
@@ -12,5 +13,5 @@
         </visual>
         <collision>
-          <origin rpy="0 0 0"/>
+          <origin rpy="0 0 0" xyz="0 0 ${disp}"/>
           <geometry>
             <mesh filename="package://sailboat_description/mesh/pt90.stl"/>
@@ -18,7 +19,7 @@
         </collision>
         <inertial>
-          <origin rpy="0 0 0" xyz="0 0 -0.05"/>
-          <mass value="0.5"/>
-          <inertia ixx="0.1" ixy="0.0" ixz="0.0" iyy="1.4" iyz="0.0" izz="1.4"/>
+          <origin rpy="0 0 0" xyz="0 0 ${disp}"/>
+          <mass value="50.0"/>
+          <inertia ixx="0.3" ixy="0.0" ixz="0.0" iyy="3.5" iyz="0.0" izz="3.6"/>
         </inertial>
     </link>
@@ -26,12 +27,12 @@
     <link name="rudder">
             <inertial>
-                <mass value="0.05" />
+                <mass value="1.0" />
                 <inertia
-                  ixx="0.05"
+                  ixx="0.0"
                   ixy="0.0"
-                  iyy="0.05"
+                  iyy="0.0"
                   ixz="0.0"
                   iyz="0.0"
-                  izz="0.005"/>
+                  izz="0.0"/>
             </inertial>
             <collision name="collision">
@@ -51,5 +52,5 @@
             <parent link="base_link"/>
             <child link="rudder"/>
-            <origin rpy="0 0 0" xyz="-0.4 0 0.0"/>
+            <origin rpy="0 0 0" xyz="-0.4 0 0"/>
             <dynamics damping="1.0"/>
             <axis xyz="0 0 1"/>
@@ -59,12 +60,12 @@
     <link name="sail">
 		<inertial>
-			<mass value="0.1" />
+			<mass value="2.0" />
 			<inertia
-			  ixx="0.4708"
+			  ixx="0.0"
 			  ixy="0.0"
-			  iyy="0.5208"
+			  iyy="0.0"
 			  ixz="0.0"
 			  iyz="0.0"
-			  izz="0.0508"/>
+			  izz="0.0"/>
 		</inertial>
 	    <collision name="collision">
@@ -84,13 +85,91 @@
         <parent link="base_link"/>
         <child link="sail"/>
-        <origin rpy="0 0 0" xyz="0.25 0 0.0"/>
+        <origin rpy="0 0 0" xyz="0.25 0 0"/>
         <dynamics damping="1.0"/>
         <axis xyz="0 0 1"/>
         <limit effort="30" velocity="5" lower="-${PI/2}" upper="${PI/2}" />
     </joint>
+<!-- KEEL DESCRIPTION -->
+    <link name="keel">
+        <inertial>
+            <mass value="10.0" xyz="0 0 0" />
+            <inertia
+              ixx="0.05"
+              ixy="0.0"
+              iyy="0.05"
+              ixz="0.0"
+              iyz="0.0"
+              izz="0.005"/>
+        </inertial>
+        <collision name="collision">
+            <geometry>
+              <mesh filename="package://sailboat_description/mesh/keel.stl"/>
+            </geometry>
+            <origin rpy="0 0 0" xyz="0 0 0"/>
+        </collision>
+        <visual name="visual">
+            <geometry>
+              <mesh filename="package://sailboat_description/mesh/keel.stl"/>
+            </geometry>
+            <origin rpy="0 0 0" xyz="0 0 0"/>
+        </visual>
+    </link>
+     <joint name="keel_joint" type="revolute">
+        <parent link="base_link"/>
+        <child link="keel"/>
+        <origin rpy="0 0 0" xyz="0 0 0"/>
+        <axis xyz="0 0 1"/>
+        <limit effort="50" velocity="0" lower="0" upper="0" />
+ 	</joint>
   <gazebo>
     <plugin name="gazebo_ros_control" filename="libgazebo_ros_control.so">
       <robotNamespace>/sailboat</robotNamespace>
     </plugin>
+	<plugin name="lifting_surface" filename="libLiftDragPlugin.so">
+    <!-- taken from the lift curve figure -->
+    <!-- alpha_0 is 5 degrees -->
+    <a0>0.08727</a0>
+    <!-- alpha_stall is 19.3 degrees -->
+    <alpha_stall>0.3368</alpha_stall>
+    <!-- slope of the lift curve to the left of the stall angle -->
+    <cla>5.418</cla>
+    <!-- slope of the lift curve to the right of the stall angle -->
+    <cla_stall>-2.1419</cla_stall>
+    <!-- below are just random values in this example -->
+    <cda>0.0</cda>
+    <cda_stall>0.0</cda_stall>
+    <cma>0.0</cma>
+    <cma_stall>0.0</cma_stall>
+    <area>3</area>
+    <fluid_density>1.2041</fluid_density>
+    <forward>-1 0 0</forward>
+    <upward>0 -1 0</upward>
+    <cp>0 0 1</cp>
+    <link_name>sail</link_name>
+    <radial_symmetry>false</radial_symmetry>
+  </plugin>
+  <plugin name="lifting_surface" filename="libLiftDragPlugin.so">
+        <!-- taken from the lift curve figure -->
+        <!-- alpha_0 is 5 degrees -->
+        <a0>0.08727</a0>
+        <!-- alpha_stall is 19.3 degrees -->
+        <alpha_stall>0.3368</alpha_stall>
+        <!-- slope of the lift curve to the left of the stall angle -->
+        <cla>5.418</cla>
+        <!-- slope of the lift curve to the right of the stall angle -->
+        <cla_stall>-2.1419</cla_stall>
+        <!-- below are just random values in this example -->
+        <cda>0.0</cda>
+        <cda_stall>0.0</cda_stall>
+        <cma>0.0</cma>
+        <cma_stall>0.0</cma_stall>
+        <area>3</area>
+        <fluid_density>1.2041</fluid_density>
+        <forward>-1 0 0</forward>
+        <upward>0 -1 0</upward>
+        <cp>0 0 1</cp>
+        <link_name>rudder</link_name>
+        <radial_symmetry>false</radial_symmetry>
+      </plugin>
   </gazebo>
   <transmission name="sail_trans">
